File: LampsBoard/ArduinoMEGAReferenceShield.brd (EAGLE design)
At the start: 101.6 x 53.3 mm, 42 parts, among them IC1 LM358N, IC2 LM358N, IC3 5V, Q1 TIP120

Commit message: Clean up
Connections:
- net VCC: now also JP3.1
Changed lines of the file:
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@@
 <wire x1="64.516" y1="28.956" x2="67.945" y2="32.385" width="0.2032" layer="1"/>
 <wire x1="64.516" y1="28.448" x2="64.516" y2="28.956" width="0.2032" layer="1"/>
-<wire x1="83.185" y1="25.4" x2="96.52" y2="50.8" width="0" layer="19" extent="1-1"/>
+<contactref element="JP3" pad="1"/>
+<wire x1="93.98" y1="50.8" x2="96.52" y2="50.8" width="0" layer="19" extent="1-1"/>
+<wire x1="83.185" y1="25.4" x2="93.98" y2="50.8" width="0" layer="19" extent="1-1"/>
 </signal>
 <signal name="D44">
