File: LampsBoard/ArduinoMEGAReferenceShield.sch (EAGLE design)
At the start: 26 parts, among them IC1 LM358N, IC2 LM358N

Commit message: Add Laser
Parts:
- added B0, B1, Z-MAX, Z-MIN: (no value), SparkFun:M02PTH
- added C9: 1uF, SparkFun:CAPPTH
- added D1: 1N4004, diode:1N4004
- added IC3: 5V, SparkFun:V_REG_78XXSIDE
- added JP8: (no value), jumper:JP3Q
- added LASER!: (no value), SparkFun:M02POLAR
- added Q1: TIP120, transistor-power:TIP120
- added R1: 10K, SparkFun:RESISTORAXIAL-0.3
- added R2: 100K, SparkFun:RESISTORAXIAL-0.3
- added R3: 1Kohm, SparkFun:RESISTORAXIAL-0.3
- added Z-AXIS: POLOLU-A4988, Pololu-A4988:POLOLU-A4988
- added Z-MOT: (no value), SparkFun:M04POLAR
- COMMUNICATION: value 14-21 (TX3 RX3 TX2 RX2 TX1 RX1 SDA) -> 14-21
Connections:
- new net A0: ADCL.1, Z-AXIS.DIR
- new net A1: ADCL.2, Z-AXIS.STEP
- new net A2: ADCL.3, R1.2, Z-AXIS.EN
- new net D44: JP2.10, Q1.B, R3.2
- new net D46: B0.1, JP2.8
- new net D48: B1.1, JP2.6
- new net D50: JP2.4, Z-MAX.1
- new net D52: JP2.2, Z-MIN.1
- new net D7: AD420ARZ1.9, PWML.8
- new net N$11: Z-AXIS.RST, Z-AXIS.SLP
- new net N$12: C9.2, IC3.OUT, LASER!.1
- new net N$13: C9.1, D1.C, LASER!.2, Q1.E
- new net N$14: Z-AXIS.GND, Z-AXIS.GND(VDD)
- new net N$15: JP8.2, R2.2, Z-AXIS.MS1
- new net N$16: JP8.4, Z-AXIS.MS2
- new net N$17: JP8.6, Z-AXIS.MS3
- new net N$20: Z-AXIS.2B, Z-MOT.1
- new net N$21: Z-AXIS.2A, Z-MOT.2
- new net N$22: Z-AXIS.1A, Z-MOT.3
- new net N$23: Z-AXIS.1B, Z-MOT.4
- new net VCC: IC3.IN, JP4.1, JP8.1, JP8.3, JP8.5, R1.1, Z-AXIS.VDD, Z-AXIS.VMOT
- net D13: now also R3.1; no longer AD420ARZ1.9
- net GND: now also B0.2, B1.2, D1.A, IC3.GND, JP5.1, JP6.1, PWMH.7, Q1.C, R2.1, Z-MAX.2, Z-MIN.2
Other:
- moved on the sheet: COMMUNICATION, JP1, JP2

Commit message: Clean up
Connections:
- net VCC: now also JP3.1
Other:
- moved on the sheet: ADCH, ADCL, B0, B1, C9, COMMUNICATION, D1, IC3, JP1, JP2, JP3, JP4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
