File: LampsBoard/LAMPS.brd (EAGLE design)
At the start: 101.6 x 53.3 mm, 42 parts, among them IC1 LM358N, IC2 LM358N, IC3 5V, Q1 TIP120

Commit message: Clean up
Parts:
- moved Z-MOT 1.27 mm to (78.1, 19.1)
Connections:
- new net D7: AD420ARZ1.9, PWML.8
- net D13: now also R3.P$1; no longer AD420ARZ1.9
- net D44: now also JP2.10; no longer R3.P$1
- net VCC: now also JP3.1
Routing:
- net D44: track 0.00 -> 108.7 mm
- net VCC: track 33.3 -> 119.5 mm
- net D7: track 0.00 -> 43.4 mm
- net N$13: track 0.00 -> 28.7 mm
- net GND: track 201.0 -> 225.5 mm
- net N$12: track 0.00 -> 15.4 mm
- net D13: track 33.4 -> 20.0 mm
- net A2: track 53.4 -> 57.2 mm
- net A0: track 45.4 -> 41.8 mm
- net N$16: track 12.5 -> 15.2 mm
- net A1: track 46.3 -> 43.9 mm
- net N$23: track 5.33 -> 6.51 mm
- net N$22: track 5.33 -> 6.51 mm
- net N$21: track 5.33 -> 6.51 mm
- net N$20: track 5.33 -> 6.51 mm
Other:
- board text added: "LASER!"

Commit message: updates
Parts:
- added C10: .33uF, SparkFun:CAP-PTH-SMALL
- added C11: 10nF, capacitor-wima:C2.5-3
- added C12, C13: 330 nF, capacitor-wima:C2.5-3
- added C14: 10 nF, capacitor-wima:C2.5-3
- added IC4, IC5: 78L12Z, linear:TO92
- C9: value 1uF -> .1uF
- moved Q1 27.7 mm to (0.64, 30.5), turned to 90 degrees
- moved D1 4.49 mm to (15.9, 46.4)
- moved R3 2.62 mm to (15.9, 41.3)
Connections:
- new net N$18: AD420ARZ.23, C1.1, C2.1, C3.1, IC4.1
- new net N$19: AD420ARZ.2, C4.2
- new net N$24: AD420ARZ1.2, C8.2
- new net N$25: AD420ARZ1.23, C5.1, C6.1, C7.1, IC5.1
- new net N$26: C13.2, C14.1, IC5.2
- net GND: now also C10.2, C11.1, C11.2, C12.2, C14.2, IC4.2; no longer AD420ARZ.2, AD420ARZ.23, AD420ARZ1.2, AD420ARZ1.23, C1.1, C2.1, C3.1, C4.2, C5.1, C6.1, C7.1, C8.2
- net VCC: now also C10.1, C12.1, C13.1, IC4.3, IC5.3
Routing:
- net GND: track 225.5 -> 0.00 mm
- net VCC: track 119.5 -> 185.4 mm
- net N$25: track 0.00 -> 60.6 mm
- net N$18: track 0.00 -> 56.9 mm
- net D11: track 32.4 -> 49.6 mm, vias 0 -> 1
- net N$26: track 0.00 -> 16.5 mm
- net D10: track 27.0 -> 10.6 mm
- net N$19: track 0.00 -> 14.1 mm
- net N$24: track 0.00 -> 13.2 mm
- net D50: track 21.6 -> 8.90 mm
- net D46: track 49.3 -> 39.3 mm
- net N$1: track 16.7 -> 24.2 mm
- net D9: track 18.0 -> 10.6 mm
- net D13: track 20.0 -> 14.5 mm
- net N$13: track 28.7 -> 32.1 mm
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- added copper zone on layer 1, net GND
- added copper zone on layer 16, net GND
