File: Lamps2.0/RAMPS_1-41.sch (EAGLE design)
At the start: 47 parts, among them Q1 STP55NF06L, Q2 STP55NF06L, U1 ARDUINO_MEGA_SHIELD, X1 MSTBA2

Commit message: Some pcb work... adding in new schematic
Parts:
- removed SER3, SER4, Z+: (no value), ultimachine:3PIN-HEADER
- removed U$2: 282837-6, RepRapjr:282837-6
- added 15V: MSTBA3, con-phoenix-508:MSTBA3
- added C1, C3, C4: 0.1uF, capacitor-wima:C2.5/2
- added C5, C7: 1uF, capacitor-wima:C2.5/2
- added GALVOX, GALVOY: (no value), ultimachine:3PIN-HEADER
- added IC2: 7805TV, linear:7805TV
- added IC3: 7906, linear:7906T
- added IC4: TLV5618, ic-package:DIL8S
- added IC5, IC6: TL082P, linear:TL082P
- added IC7: 7806TV, linear:7805TV
- added R1: 20k, pot:TRIM_US-B25P
- added R11, R15, R16, R17: 10k, adafruit:R-US_R0805
- added R18, R19, R23, R26: 200k, adafruit:R-US_R0805
- added R3, R4: 1k, pot:TRIM_US-B25P
- added R5, R6, R7, R8: 100k, adafruit:R-US_R0805
- added U$1, U$4: THAT1646, THAT1646:THAT1646
- added X2: MSTBA4, con-phoenix-508:MSTBA4
Connections:
- removed net Y-MAX: U1.D15
- removed net Y-MIN: U1.D14
- new net D14: IC4.1, U1.D14
- new net D15: IC4.2, U1.D15
- new net GND_0: 15V-3.1, C1.2, C3.2, C4.2, GALVOX.3, GALVOY.3, IC2.GND, IC3.GND, IC4.5, IC7.GND, R1.E, R11.2, R16.2, R23.1, R26.1, U$1.GND, U$4.GND
- new net N$10: IC6B.+IN, R4.S
- new net N$11: IC5B.+IN, R3.S
- new net N$12: GALVOX.2, U$1.OUT-, U$1.SNS-
- new net N$13: GALVOX.1, U$1.OUT+, U$1.SNS+
- new net N$14: IC5B.-IN, IC5B.OUT, R5.2
- new net N$15: IC5A.-IN, R18.2, R5.1
- new net N$16: IC4.7, R7.2
- new net N$17: IC5A.+IN, R26.2, R7.1
- new net N$18: IC6B.-IN, IC6B.OUT, R6.2
- new net N$2: 15V-1.1, IC2.VI, IC7.VI
- new net N$20: IC6A.-IN, R19.2, R6.1
- new net N$21: IC4.4, R8.2
- new net N$22: IC6A.+IN, R23.2, R8.1
- new net N$24: GALVOY.2, U$4.OUT-, U$4.SNS-
- new net N$25: GALVOY.1, U$4.OUT+, U$4.SNS+
- new net N$3: 15V-2.1, IC3.VI
- new net N$4: R16.1, R4.A
- new net N$5: R17.2, R4.E
- new net N$6: IC4.6, R1.S
- new net N$8: R11.1, R3.A
- new net N$9: R15.2, R3.E
- new net NEG_6V: C4.1, C5.1, IC3.VO, IC5P.V-, IC6P.V-, U$1.V-
- new net POS_5V: C1.1, IC2.VO, IC4.8, R1.A, R15.1, R17.1
- new net POS_6V: C3.1, C7.1, IC5P.V+, IC6P.V+, IC7.VO, U$1.V+
- new net T2_5: C5.2, U$4.V-
- new net T2_6: C7.2, U$4.V+
- new net X_IN: IC5A.OUT, R18.1, U$1.IN
- new net Y_IN: IC6A.OUT, R19.1, U$4.IN
- net +12V: now also X2-1.1, X2-3.1; no longer U$2.P$3, U$2.P$5
- net +5V: no longer SER3.2, SER4.2
- net D16: now also IC4.3; no longer U$9.18
- net D17: no longer U$9.17
- net D4: no longer SER4.3
- net D5: no longer SER3.3
- net GND: no longer SER3.1, SER4.1, Z+.2
- net N$1: now also X2-2.1; no longer U$2.P$4
- net N$7: now also X2-4.1; no longer U$2.P$6
- net VCC: no longer Z+.3
- net Z-MAX: no longer Z+.1
Other:
- note added: "+/- 15V Power"
- note added: "12V Power"
- note added: "Copyright 2012 Justin Hawkins"
- note added: "GND from PS"
- note added: "Hawkinsoft LLC"
- note added: "LAMPS 0.1 (Laser Arduino Mega Pololu Shield)"
- note added: "Neg 15V from PS"
- note added: "Pos 15V from PS"
- note added: "X-Neg"
- note added: "X-Pos"
- note added: "Y-Neg"
- note added: "Y-Pos"
- note removed: "Copyright 2011 Johnny Russell"
- note removed: "Power"
- note removed: "RAMPS 1.4 (RepRap Arduino Mega Pololu Shield)"
- note removed: "UltiMachine"
- note removed: "reprap.org/wiki/RAMPS1.4"
- moved on the sheet: C10
