File: Lamps2.0/LAMPS_1-41.sch (EAGLE design)
At the start: 82 parts, among them IC2 7805TV, IC4 TLV5618, IC5 TL082P, IC6 TL082P, IC7 7806TV, Q1 STP55NF06L, Q2 STP55NF06L, U1 ARDUINO_MEGA_SHIELD, X1 MSTBA2, X2 MSTBA4

Commit message: Shuffle Board, Gen Gerbers
Parts:
- renumbered X1 to 12V, X2 to 12VOUT
Changed lines of the file:
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@@
 <part name="P+49" library="supply1" deviceset="+12V" device=""/>
 <part name="GND39" library="supply1" deviceset="GND" device=""/>
-<part name="X1" library="con-phoenix-508" deviceset="MSTBA2" device=""/>
-<part name="X2" library="con-phoenix-508" deviceset="MSTBA4" device=""/>
+<part name="12V" library="con-phoenix-508" deviceset="MSTBA2" device=""/>
+<part name="12VOUT" library="con-phoenix-508" deviceset="MSTBA4" device=""/>
 <part name="IC4" library="ic-package" deviceset="DIL8" device="S" value="TLV5618"/>
 <part name="R1" library="pot" deviceset="TRIM_US-" device="B25P" value="20k"/>
@@
 <instance part="P+49" gate="1" x="-129.54" y="48.26"/>
 <instance part="GND39" gate="1" x="-129.54" y="40.64"/>
-<instance part="X1" gate="-1" x="-180.34" y="55.88"/>
-<instance part="X1" gate="-2" x="-180.34" y="48.26"/>
-<instance part="X2" gate="-1" x="-129.54" y="127" rot="R180"/>
-<instance part="X2" gate="-2" x="-129.54" y="132.08" rot="R180"/>
-<instance part="X2" gate="-3" x="-129.54" y="137.16" rot="R180"/>
-<instance part="X2" gate="-4" x="-129.54" y="142.24" rot="R180"/>
+<instance part="12V" gate="-1" x="-180.34" y="55.88"/>
+<instance part="12V" gate="-2" x="-180.34" y="48.26"/>
+<instance part="12VOUT" gate="-1" x="-129.54" y="127" rot="R180"/>
+<instance part="12VOUT" gate="-2" x="-129.54" y="132.08" rot="R180"/>
+<instance part="12VOUT" gate="-3" x="-129.54" y="137.16" rot="R180"/>
+<instance part="12VOUT" gate="-4" x="-129.54" y="142.24" rot="R180"/>
 <instance part="IC4" gate="G$1" x="-81.28" y="177.8"/>
 <instance part="R1" gate="G$1" x="-58.42" y="175.26" rot="R180"/>
@@
 <pinref part="GND14" gate="1" pin="GND"/>
 <pinref part="D2" gate="1" pin="A"/>
-<pinref part="X1" gate="-2" pin="1"/>
+<pinref part="12V" gate="-2" pin="1"/>
 </segment>
 <segment>
@@
 <pinref part="R24" gate="G$1" pin="1"/>
 <pinref part="R25" gate="G$1" pin="1"/>
-<pinref part="X2" gate="-3" pin="1"/>
-<pinref part="X2" gate="-1" pin="1"/>
+<pinref part="12VOUT" gate="-3" pin="1"/>
+<pinref part="12VOUT" gate="-1" pin="1"/>
 </segment>
 <segment>
@@
 <pinref part="Q2" gate="1" pin="D"/>
 <pinref part="LED3" gate="G$1" pin="C"/>
-<pinref part="X2" gate="-2" pin="1"/>
+<pinref part="12VOUT" gate="-2" pin="1"/>
 </segment>
 </net>
@@
 <pinref part="Q1" gate="1" pin="D"/>
 <pinref part="LED4" gate="G$1" pin="C"/>
-<pinref part="X2" gate="-4" pin="1"/>
+<pinref part="12VOUT" gate="-4" pin="1"/>
 </segment>
 </net>
@@
 <wire x1="-175.26" y1="55.88" x2="-162.56" y2="55.88" width="0.1524" layer="91"/>
 <pinref part="F1" gate="A" pin="2"/>
-<pinref part="X1" gate="-1" pin="1"/>
-</segment>
-</net>
+<pinref part="12V" gate="-1" pin="1"/>
+</segment>
+</net>
