File: Lamps2.0/LAMPS_1-41.brd (EAGLE design)
At the start: 101.6 x 60.3 mm, 82 parts, among them IC2 7805TV, IC4 TLV5618, IC5 TL082P, IC6 TL082P, IC7 7806TV, Q1 STP55NF06L, Q2 STP55NF06L, U1 ARDUINO_MEGA_SHIELD, X1 MSTBA2, X2 MSTBA4

Commit message: Start relaying board
Parts:
- moved SER1 196.2 mm to (16.5, -128.3), turned to 0 degrees
- moved LED4 188.4 mm to (30.5, -121.9), turned to 0 degrees
- moved R25 188.4 mm to (66.0, -114.3), turned to 0 degrees
- moved LED3 188.1 mm to (25.4, -121.9), turned to 0 degrees
- moved LED1 186.7 mm to (20.3, -121.9)
- moved R24 185.8 mm to (59.7, -114.3), turned to 0 degrees
- moved R20 184.6 mm to (-6.35, -120.7)
- moved R6 183.8 mm to (-10.2, -114.3), turned to 0 degrees
- moved R13 180.7 mm to (77.5, -114.3), turned to 0 degrees
- moved R12 178.9 mm to (72.4, -114.3)
- moved 12V-AUX 177.3 mm to (34.3, -120.7)
- moved R5 171.8 mm to (-16.5, -114.3), turned to 0 degrees
- moved R10 171.4 mm to (15.2, -114.3), turned to 0 degrees
- moved R27 170.3 mm to (-1.27, -120.7)
- moved R29 166.0 mm to (-7.62, -86.4)
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Connections:
- removed net E1-DIR: U1.D34
- removed net E1-STEP: U1.D36
- removed net X-EN: U1.D38
- new net D34: BUTTONS.5, U1.D34
- new net D36: BUTTONS.3, U1.D36
- new net D38: BUTTONS.1, U1.D38
- net D23: no longer BUTTONS.1
- net D25: no longer BUTTONS.3
- net D27: no longer BUTTONS.5
- net D29: no longer BUTTONS.7
- net D32: now also BUTTONS.7
Routing:
- net VCC: track 339.4 -> 0.00 mm, vias 11 -> 0
- net POS_5V: track 162.6 -> 0.00 mm, vias 9 -> 0
- net D2: track 135.1 -> 0.00 mm, vias 10 -> 0
- net D43: track 121.4 -> 0.00 mm, vias 5 -> 0
- net D23: track 117.1 -> 0.00 mm, vias 5 -> 0
- net +12V: track 116.9 -> 0.00 mm, vias 1 -> 0
- net POS_6V: track 113.6 -> 0.00 mm, vias 3 -> 0
- net D12: track 109.8 -> 0.00 mm, vias 2 -> 0
- net N$24: track 105.0 -> 0.00 mm, vias 3 -> 0
- net N$12: track 98.1 -> 0.00 mm, vias 6 -> 0
- net D1: track 91.5 -> 0.00 mm, vias 5 -> 0
- net N$25: track 90.0 -> 0.00 mm, vias 4 -> 0
- net NEG_6V: track 90.0 -> 0.00 mm, vias 1 -> 0
- net Z-STEP: track 88.3 -> 0.00 mm, vias 3 -> 0
- net N$6: track 79.4 -> 0.00 mm, vias 3 -> 0
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- removed copper zone on layer 1, net GND
- removed copper zone on layer 1, net GND_0
- removed copper zone on layer 16, net GND_0
Other:
- board text removed: "10"
- board text removed: "1A"
- board text removed: "1B"
- board text removed: "2A"
- board text removed: "2B"
- board text removed: "8"
- board text removed: "9"
- board text removed: "AUX-3"
- board text removed: "Copyright 2011 Johnny Russell - UltiMachine"
- board text removed: "END STOPS"
- board text removed: "MS3"
- board text removed: "PS"
- board text removed: "RESET"
- board text removed: "SERVOS"
- board text removed: "Z"
- board text removed: "s"

Commit message: Shuffle Board, Gen Gerbers
Parts:
- added U$2: (no value), ohw-logo:OSHW_FILLX1000_NOTEXT
- moved R27 202.6 mm to (100.3, 54.6), turned to 270 degrees
- moved TTL 202.3 mm to (100.3, 36.8), turned to 180 degrees
- moved R28 195.6 mm to (100.3, 49.5), turned to 90 degrees
- moved 5V 195.0 mm to (40.6, 59.7), turned to 180 degrees
- moved LEDA 186.6 mm to (100.3, 62.2), turned to 270 degrees
- moved R20 184.5 mm to (87.6, 38.1), turned to 90 degrees
- moved SER1 184.0 mm to (36.8, 54.6), turned to 180 degrees
- moved VCC 180.8 mm to (50.8, 57.1), turned to 270 degrees
- moved SERIAL 179.4 mm to (58.4, 50.8)
- moved R8 177.1 mm to (47.0, 57.1)
- moved R12 175.6 mm to (29.2, 55.9), turned to 90 degrees
- moved R11 173.6 mm to (43.2, 49.5)
- moved GALVOX 172.8 mm to (1.27, 44.5), turned to 270 degrees
- moved R7 172.8 mm to (67.3, 43.2)
- moved LED1 171.7 mm to (29.2, 49.5), turned to 180 degrees
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- renumbered X1 to 12V, X2 to 12VOUT
Routing:
- net GND_0: track 0.00 -> 240.5 mm, vias 0 -> 3
- net VCC: track 0.00 -> 227.0 mm, vias 0 -> 4
- net N$8: track 0.00 -> 181.9 mm
- net +12V: track 0.00 -> 147.4 mm, vias 0 -> 2
- net D9: track 0.00 -> 111.3 mm, vias 0 -> 2
- net N$2: track 0.00 -> 92.1 mm
- net POS_6V: track 0.00 -> 91.3 mm, vias 0 -> 1
- net NEG_6V: track 0.00 -> 82.2 mm, vias 0 -> 3
- net POS_5V: track 0.00 -> 81.9 mm, vias 0 -> 1
- net A4: track 0.00 -> 80.3 mm, vias 0 -> 1
- net Z-DIR: track 0.00 -> 66.8 mm, vias 0 -> 2
- net Y_IN: track 0.00 -> 64.0 mm, vias 0 -> 2
- net D37: track 0.00 -> 62.9 mm, vias 0 -> 2
- net N$6: track 0.00 -> 60.9 mm
- net N$7: track 0.00 -> 59.3 mm, vias 0 -> 2
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- added copper zone on layer 1, net GND
- added copper zone on layer 16, net GND
- added copper zone on layer 1, net GND_0
- added copper zone on layer 16, net GND_0
Other:
- outline, holes or cut-outs redrawn
- board text added: "C 2012 Hawkinsoft LLC - Lamps 1.0"
- board text added: "G"

Commit message: LAMPS 1.0 GERBERS
Parts:
- moved LED4 33.4 mm to (13.8, 11.6)
- moved R15 30.2 mm to (79.8, 53.2), turned to 180 degrees
- moved R26 17.6 mm to (65.8, 43.1), turned to 270 degrees
- moved R10 11.7 mm to (54.4, 52.3), turned to 0 degrees
- moved C7 10.9 mm to (18.5, 46.7)
- moved R16 7.37 mm to (5.33, 33.3)
- moved R18 7.06 mm to (21.8, 41.7), turned to 0 degrees
- moved R19 6.93 mm to (24.9, 34.5)
- moved C5 6.75 mm to (24.9, 56.3)
- moved U$1 6.55 mm to (11.6, 46.2)
- moved D1 6.41 mm to (28.3, 25.4)
- moved R9 6.01 mm to (38.2, 55.1), turned to 180 degrees
- moved R11 5.70 mm to (48.8, 50.7)
- moved R2 5.27 mm to (17.8, 21.5)
- moved SERIAL 5.21 mm to (58.2, 56.0)
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Routing:
- net N$8: track 181.9 -> 53.5 mm, vias 0 -> 2
- net GND_0: track 240.5 -> 163.5 mm, vias 3 -> 4
- net N$2: track 92.1 -> 51.5 mm, vias 0 -> 1
- net A4: track 80.3 -> 46.2 mm, vias 1 -> 3
- net D9: track 111.3 -> 90.1 mm, vias 2 -> 1
- net N$9: track 52.5 -> 73.3 mm
- net POS_6V: track 91.3 -> 72.6 mm, vias 1 -> 2
- net Y_IN: track 64.0 -> 45.5 mm, vias 2 -> 1
- net T2_5: track 14.3 -> 31.0 mm, vias 0 -> 1
- net N$40: track 26.3 -> 42.6 mm, vias 1 -> 2
- net N$22: track 48.9 -> 34.8 mm, vias 3 -> 0
- net D39: track 36.5 -> 49.9 mm, vias 1 -> 2
- net POS_5V: track 81.9 -> 92.7 mm, vias 1 -> 2
- net NEG_6V: track 82.2 -> 92.5 mm
- net D37: track 62.9 -> 53.2 mm, vias 2 -> 4
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Other:
- outline, holes or cut-outs redrawn

Commit message: Clean-Up, Add Top Z Mount
Parts:
- moved U$2 9.94 mm to (94.2, 40.1)
- moved GALVOX 1.85 mm to (3.05, 45.0)
- moved GALVOY 1.78 mm to (3.05, 35.6)
- moved LCD 1.05 mm to (94.2, 13.0)
- moved LEDA 1.02 mm to (99.3, 62.2)
- moved LEDB 1.02 mm to (99.3, 41.9)
- moved TTL 1.02 mm to (99.3, 36.8)
- moved R16 0.92 mm to (6.10, 32.8)
- moved R27 0.76 mm to (99.6, 54.6)
- moved R28 0.76 mm to (99.6, 49.5)
Routing:
- net D35: track 35.9 -> 74.1 mm, vias 0 -> 1
- net N$7: track 59.1 -> 89.7 mm, vias 3 -> 1
- net Z-DIR: track 63.4 -> 34.7 mm, vias 2 -> 1
- net VCC: track 224.5 -> 196.1 mm, vias 0 -> 2
- net D9: track 90.1 -> 69.3 mm
- net POS_5V: track 92.7 -> 112.2 mm, vias 2 -> 0
- net D37: track 53.2 -> 36.4 mm, vias 4 -> 0
- net Z-MAX: track 23.6 -> 36.7 mm, vias 1 -> 0
- net T2_5: track 31.0 -> 20.1 mm
- net MOSI: track 18.8 -> 8.67 mm, vias 1 -> 0
- net N$4: track 65.1 -> 55.1 mm
- net D39: track 49.9 -> 40.8 mm, vias 2 -> 1
- net SCK: track 16.6 -> 8.67 mm
- net N$9: track 73.3 -> 65.4 mm
- net +12V: track 142.5 -> 135.4 mm
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Other:
- board size 101.6 x 60.3 mm -> 99.8 x 60.3 mm
