File: Lamps2.0/LAMPS.sch (EAGLE design)
At the start: 82 parts, among them IC2 7805TV, IC4 TLV5618, IC5 TL082P, IC6 TL082P, IC7 7806TV, Q1 STP55NF06L, Q2 STP55NF06L, U1 ARDUINO_MEGA_SHIELD

Commit message: Making strides
Parts:
- removed R27: 1K, adafruit:R-US_R0805
Connections:
- removed net N$19: LEDA.1, R27.1
- net D31: no longer R27.2
Changed lines of the file:
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@@
-<attribute name="OC_NEWARK" value="unknown"/>
-</part>
-<part name="R27" library="adafruit" deviceset="R-US_" device="R0805" value="1K">
-<attribute name="MF" value=""/>
-<attribute name="MPN" value=""/>
 <attribute name="OC_NEWARK" value="unknown"/>
 </part>
@@
 <attribute name="MPN" x="-78.74" y="210.82" size="1.778" layer="96" display="off"/>
 </instance>
-<instance part="R27" gate="G$1" x="-96.52" y="228.6" rot="R180">
-<attribute name="OC_NEWARK" x="-96.52" y="228.6" size="1.778" layer="96" display="off"/>
-<attribute name="MF" x="-96.52" y="228.6" size="1.778" layer="96" display="off"/>
-<attribute name="MPN" x="-96.52" y="228.6" size="1.778" layer="96" display="off"/>
-</instance>
 <instance part="R28" gate="G$1" x="-96.52" y="210.82" rot="R180">
 <attribute name="OC_NEWARK" x="-96.52" y="210.82" size="1.778" layer="96" display="off"/>
@@
 </segment>
 <segment>
-<pinref part="R27" gate="G$1" pin="2"/>
-<wire x1="-101.6" y1="228.6" x2="-104.14" y2="228.6" width="0.1524" layer="91"/>
+<wire x1="-86.36" y1="228.6" x2="-104.14" y2="228.6" width="0.1524" layer="91"/>
 <label x="-104.14" y="228.6" size="1.778" layer="95" rot="R180" xref="yes"/>
 </segment>
@@
 </segment>
 </net>
-<net name="N$19" class="0">
-<segment>
-<pinref part="R27" gate="G$1" pin="1"/>
-<pinref part="LEDA" gate="G$1" pin="1"/>
-<wire x1="-91.44" y1="228.6" x2="-86.36" y2="228.6" width="0.1524" layer="91"/>
-</segment>
-</net>
