File: Lamps2.1/LAMPS.brd (EAGLE design)
At the start: 99.8 x 60.3 mm, 104 parts, among them IC2 7805TV, IC4 TLV5618, IC5 TL082P, IC6 TL082P, IC7 7806TV, Q1 STP55NF06L, Q2 STP55NF06L, U1 ARDUINO_MEGA_SHIELD

Commit message: Nightly Commit ... laser moves much better... more work to be done on planner
Parts:
- removed 12V-AUX: (no value), SparkFun:1X02
- removed R46, R47, R48: 10k, adafruit:R0805
- removed U$2: (no value), ohw-logo:OSHW_FILLX1000_NOTEXT
- removed VCC: (no value), adafruit:1X01
- moved R53 254.4 mm to (54.9, 76.2), turned to 90 degrees
- moved R52 249.8 mm to (57.4, 76.2), turned to 90 degrees
- moved R51 245.2 mm to (59.9, 76.2), turned to 90 degrees
- moved R59 244.4 mm to (33.5, 22.9), turned to 180 degrees
- moved R58 241.7 mm to (33.5, 25.7), turned to 180 degrees
- moved R50 240.7 mm to (62.5, 76.2), turned to 90 degrees
- moved TFT01-3.2 239.5 mm to (26.9, 43.9), turned to 270 degrees
- moved R57 239.5 mm to (33.5, 29.0), turned to 180 degrees
- moved R49 236.3 mm to (65.0, 76.2), turned to 90 degrees
- moved R60 236.1 mm to (3.81, 20.8), turned to 270 degrees
- moved R55 232.6 mm to (33.8, 47.8), turned to 180 degrees
- moved R56 230.6 mm to (33.8, 40.1), turned to 180 degrees
- moved R54 224.6 mm to (33.8, 45.2), turned to 180 degrees
- moved R45 205.2 mm to (83.1, 56.4), turned to 180 degrees
- moved R44 202.3 mm to (89.2, 55.1), flipped to the bottom, turned to 180 degrees
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Connections:
- removed net N$57: R46.1, U1.D51
- removed net N$58: R47.1, U1.D52
- removed net N$59: R48.1, U1.D53
- net +12V: no longer 12V-AUX.1
- net D12: now also LEDA.1
- net GND: no longer 12V-AUX.2
- net SD_CS: now also U1.D53; no longer R48.2
- net SD_IN: now also U1.D51; no longer R46.2
- net SD_SCK: now also U1.D52; no longer R47.2
- net VCC: no longer VCC.1
- net Z-DIR: now also U1.D14; no longer U1.D15
- net Z-STEP: now also U1.D15; no longer U1.D14
Routing:
- added copper zone on layer 1, net GND
- added copper zone on layer 16, net VCC
Other:
- board size 99.8 x 60.3 mm -> 99.8 x 75.6 mm
- board text removed: "+"
- board text removed: "-"
- board text removed: "1"
- board text removed: "AUX-4"
- board text removed: "C 2012 Hawkinsoft LLC - Lamps 1.0"
- board text removed: "G"

Commit message: Updates to 2.1 Board
Parts:
- removed Z+, Z-: (no value), ultimachine:3PIN-HEADER
- added ZMAX, ZMIN: (no value), SparkFun:1X02
- moved 2.048V 67.3 mm to (25.7, 70.6), turned to 0 degrees
- moved IC4 59.5 mm to (27.9, 60.7), turned to 90 degrees
- moved R8 57.5 mm to (20.3, 70.1)
- moved R24 55.0 mm to (72.6, 28.2), turned to 90 degrees
- moved R16 51.7 mm to (20.6, 52.6), turned to 90 degrees
- moved R7 50.2 mm to (20.1, 64.5), turned to 270 degrees
- moved R15 49.1 mm to (20.3, 22.6)
- moved R17 48.0 mm to (36.8, 66.0), turned to 180 degrees
- moved R4 47.6 mm to (26.9, 49.0)
- moved R3 42.2 mm to (26.9, 26.7)
- moved R26 41.9 mm to (6.35, 30.2)
- moved R11 40.2 mm to (26.4, 19.1), turned to 270 degrees
- moved R56 38.5 mm to (47.2, 76.2), turned to 90 degrees
- moved R54 36.1 mm to (52.3, 76.2), turned to 90 degrees
- moved TFT01-3.2 34.8 mm to (61.7, 43.7), turned to 0 degrees
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Connections:
- net GND: now also ZMAX.2, ZMIN.2; no longer Z+.2, Z-.2
- net VCC: no longer Z+.3, Z-.3
- net Z-MAX: now also ZMAX.1; no longer Z+.1
- net Z-MIN: now also ZMIN.1; no longer Z-.1
Routing:
- net N$23: track 0.00 -> 267.3 mm, vias 0 -> 4
- net DB13: track 0.00 -> 206.5 mm, vias 0 -> 6
- net DB14: track 0.00 -> 166.7 mm, vias 0 -> 6
- net D19: track 0.00 -> 161.5 mm, vias 0 -> 1
- net DB12: track 0.00 -> 154.9 mm, vias 0 -> 3
- net POS_6V: track 0.00 -> 148.7 mm, vias 0 -> 2
- net DB15: track 0.00 -> 141.9 mm, vias 0 -> 6
- net CS: track 0.00 -> 138.0 mm, vias 0 -> 7
- net SD_SCK: track 0.00 -> 136.9 mm, vias 0 -> 7
- net +12V: track 0.00 -> 134.5 mm
- net POS_5V: track 0.00 -> 133.3 mm, vias 0 -> 2
- net DB11: track 0.00 -> 119.0 mm, vias 0 -> 8
- net SD_OUT: track 0.00 -> 113.0 mm, vias 0 -> 4
- net NEG_6V: track 0.00 -> 110.6 mm, vias 0 -> 3
- net RS: track 0.00 -> 109.4 mm, vias 0 -> 2
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
Commit message: Updated boards
Parts:
- removed 12V: MSTBA3, con-phoenix-508:MSTBA3
- removed IC4: TLV5618, ic-package:SOCKET-08
- removed IC5, IC6: TL082P, linear:DIL08
- added !!!SCHEMATICDOESNOTREFLECTDESIGN1: 7912, linear:TO220V
- added 15V: MSTBA3, con-phoenix-508:MSTBA3
- added IC1: 7812TV, linear:TO220V
- added TL082D-1, TL082D-2: TL082D, linear:SO08
- added U$2: THAT1646SMD, TLV5618:TLV5618
- added U$3: (no value), ohw-logo:OSHW_FILLX350_NOTEXT
- moved LED1 5.49 mm to (21.3, 80.5)
- moved U$1 5.24 mm to (7.87, 49.5)
- moved U$4 5.24 mm to (8.13, 60.2)
- moved R37 5.09 mm to (89.4, 63.8)
- moved R43 5.08 mm to (89.4, 55.4)
- moved R36 4.82 mm to (88.9, 62.5)
- moved R42 4.58 mm to (88.9, 55.1)
- moved R12 3.30 mm to (26.2, 74.7)
- moved C3 3.06 mm to (51.3, 27.7)
- moved !!!SCHEMATICDOESNOTREFLECTDESIGN 2.84 mm to (42.4, 13.5)
- moved R38 2.50 mm to (88.9, 59.7)
- moved C1 2.30 mm to (68.3, 27.9)
- moved 2.048V 1.55 mm to (25.9, 69.1)
- moved IC7 1.44 mm to (54.4, 24.1)
- moved TFT01-3.2 1.44 mm to (60.7, 44.7), turned to 180 degrees
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- renumbered LEDA to LASER
Connections:
- new net N$58: 15V.1, IC1.1
- new net N$59: !!!SCHEMATICDOESNOTREFLECTDESIGN1.2, 15V.2
- net D20: now also U$2.3; no longer IC4.3
- net GND: now also !!!SCHEMATICDOESNOTREFLECTDESIGN1.1, 15V.3, IC1.2, U$2.5; no longer 12V.3, IC4.5
- net N$10: now also TL082D-2.5; no longer IC6.5
- net N$11: now also TL082D-1.5; no longer IC5.5
- net N$14: now also TL082D-1.6, TL082D-1.7; no longer IC5.6, IC5.7
- net N$15: now also TL082D-1.2; no longer IC5.2
- net N$16: now also U$2.7; no longer IC4.7
- net N$17: now also TL082D-1.3; no longer IC5.3
- net N$18: now also TL082D-2.6, TL082D-2.7; no longer IC6.6, IC6.7
- net N$20: now also TL082D-2.2; no longer IC6.2
- net N$21: now also U$2.4; no longer IC4.4
- net N$22: now also TL082D-2.3; no longer IC6.3
- net N$3: now also !!!SCHEMATICDOESNOTREFLECTDESIGN1.3; no longer 12V.2
- net N$6: now also U$2.6; no longer IC4.6
- net NEG_6V: now also TL082D-1.4, TL082D-2.4; no longer IC5.4, IC6.4
- net POS_12V: now also IC1.3; no longer 12V.1
- net POS_5V: now also U$2.8; no longer IC4.8
- net POS_6V: now also TL082D-1.8, TL082D-2.8; no longer IC5.8, IC6.8
- net SD_IN: now also U$2.1; no longer IC4.1
- net SD_SCK: now also U$2.2; no longer IC4.2
- net X_IN: now also TL082D-1.1; no longer IC5.1
- net Y_IN: now also TL082D-2.1; no longer IC6.1
Routing:
- net N$23: track 267.3 -> 0.00 mm, vias 4 -> 0
- net DB13: track 206.5 -> 0.00 mm, vias 6 -> 0
- net DB14: track 166.7 -> 0.00 mm, vias 6 -> 0
- net D19: track 161.5 -> 0.00 mm, vias 1 -> 0
- net DB12: track 154.9 -> 0.00 mm, vias 3 -> 0
- net POS_6V: track 148.7 -> 0.00 mm, vias 2 -> 0
- net DB15: track 141.9 -> 0.00 mm, vias 6 -> 0
- net CS: track 138.0 -> 0.00 mm, vias 7 -> 0
- net SD_SCK: track 136.9 -> 0.00 mm, vias 7 -> 0
- net +12V: track 134.5 -> 0.00 mm
- net POS_5V: track 133.3 -> 0.00 mm, vias 2 -> 0
- net DB11: track 119.0 -> 0.00 mm, vias 8 -> 0
- net SD_OUT: track 113.0 -> 0.00 mm, vias 4 -> 0
- net NEG_6V: track 110.6 -> 0.00 mm, vias 3 -> 0
- net RS: track 109.4 -> 0.00 mm, vias 2 -> 0
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- added copper zone on layer 16, net GND
- removed copper zone on layer 16, net VCC
Other:
- board text added: "+ - GND"
- board text added: "2013 c (GPL)"
- board text added: "7805"
- board text added: "7806"
- board text added: "7812"
- board text added: "7906"
- board text added: "7912"
- board text added: "LAMPS 2.1"
- board text added: "LAMPS 2.1 (Laser Arduino MEGA Pololu Shield)"
- board text added: "STP55"
- board text added: "prYntech"
- board text removed: "LAMPS 0.1 (Laser Arduino MEGA Pololu Shield)"
