File: Lamps2.1/LAMPS.sch (EAGLE design)
At the start: 103 parts, among them IC2 7805TV, IC4 TLV5618, IC5 TL082P, IC6 TL082P, IC7 7806TV, Q1 STP55NF06L, Q2 STP55NF06L, U1 ARDUINO_MEGA_SHIELD

Commit message: Nightly Commit ... laser moves much better... more work to be done on planner
Parts:
- removed 12V-AUX: (no value), SparkFun:M02PTH
- removed R46, R47, R48: 10k, adafruit:R-US_R0805
- removed VCC: (no value), adafruit:PINHD-1X1
Connections:
- removed net N$57: R46.1, U1.D51
- removed net N$58: R47.1, U1.D52
- removed net N$59: R48.1, U1.D53
- net +12V: no longer 12V-AUX.1
- net D12: now also LEDA.1
- net GND: no longer 12V-AUX.2
- net SD_CS: now also U1.D53; no longer R48.2
- net SD_IN: now also U1.D51; no longer R46.2
- net SD_SCK: now also U1.D52; no longer R47.2
- net VCC: no longer VCC.1
- net Z-DIR: now also U1.D14; no longer U1.D15
- net Z-STEP: now also U1.D15; no longer U1.D14
Other:
- moved on the sheet: !!~{SCHEMATICDOESNOTREFLECTDESIGN}, 12V-1, 12V-2, 12V-3, 12VOUT-1, 12VOUT-2, 12VOUT-3, 12VOUT-4, 2.048V, 2.5V, 2.5VY, C1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

Commit message: Updates to 2.1 Board
Parts:
- removed Z+, Z-: (no value), ultimachine:3PIN-HEADER
- added ZMAX, ZMIN: (no value), SparkFun:M02PTH
Connections:
- net GND: now also ZMAX.2, ZMIN.2; no longer Z+.2, Z-.2
- net VCC: no longer Z+.3, Z-.3
- net Z-MAX: now also ZMAX.1; no longer Z+.1
- net Z-MIN: now also ZMIN.1; no longer Z-.1

Commit message: Updated boards
Parts:
- removed 12V: MSTBA3, con-phoenix-508:MSTBA3
- removed IC4: TLV5618, ic-package:DIL8S
- removed IC5, IC6: TL082P, linear:TL082P
- removed LEDA: (no value), SparkFun:M02PTH
- added !!!SCHEMATICDOESNOTREFLECTDESIGN1: 7912, linear:7805TV
- added 15V: MSTBA3, con-phoenix-508:MSTBA3
- added IC1: 7812TV, linear:7812TV
- added LASER: (no value), SparkFun:M02PTH
- added TL082D-1, TL082D-2: TL082D, linear:TL082D
- added U$2: THAT1646SMD, TLV5618:THAT1646SMD
Connections:
- new net N$58: 15V-1.1, IC1.VI
- new net N$59: !!!SCHEMATICDOESNOTREFLECTDESIGN1.GND, 15V-2.1
- net D12: now also LASER.1; no longer LEDA.1
- net D20: now also U$2.CS; no longer IC4.3
- net GND: now also !!!SCHEMATICDOESNOTREFLECTDESIGN1.VI, 15V-3.1, IC1.GND, LASER.2, U$2.GND; no longer 12V-3.1, IC4.5, LEDA.2
- net N$10: now also TL082D-2B.+IN; no longer IC6B.+IN
- net N$11: now also TL082D-1B.+IN; no longer IC5B.+IN
- net N$14: now also TL082D-1B.-IN, TL082D-1B.OUT; no longer IC5B.-IN, IC5B.OUT
- net N$15: now also TL082D-1A.-IN; no longer IC5A.-IN
- net N$16: now also U$2.OUTB; no longer IC4.7
- net N$17: now also TL082D-1A.+IN; no longer IC5A.+IN
- net N$18: now also TL082D-2B.-IN, TL082D-2B.OUT; no longer IC6B.-IN, IC6B.OUT
- net N$20: now also TL082D-2A.-IN; no longer IC6A.-IN
- net N$21: now also U$2.OUTA; no longer IC4.4
- net N$22: now also TL082D-2A.+IN; no longer IC6A.+IN
- net N$3: now also !!!SCHEMATICDOESNOTREFLECTDESIGN1.VO; no longer 12V-2.1
- net N$6: now also U$2.REF; no longer IC4.6
- net NEG_6V: now also TL082D-1P.V-, TL082D-2P.V-; no longer IC5P.V-, IC6P.V-
- net POS_12V: now also IC1.VO; no longer 12V-1.1
- net POS_5V: now also U$2.VDD; no longer IC4.8
- net POS_6V: now also TL082D-1P.V+, TL082D-2P.V+; no longer IC5P.V+, IC6P.V+
- net SD_IN: now also U$2.DIN; no longer IC4.1
- net SD_SCK: now also U$2.SCLK; no longer IC4.2
- net X_IN: now also TL082D-1A.OUT; no longer IC5A.OUT
- net Y_IN: now also TL082D-2A.OUT; no longer IC6A.OUT
Other:
- note added: "+/- 15V Power"
- note added: "Neg 15V from PS"
- note added: "Pos 15V from PS"
- note added: "X&Y Galvos"
- note added: "prYntech 2013 (c) GPL"
- note removed: "+/- 12V Power"
- note removed: "Neg 12V from PS"
- note removed: "Pos 12V from PS"
- moved on the sheet: 2.048V, C2, C6, D1, D2, F1, R57, R58, R59, R60, S1, TFT01-3.2-1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
